File: digital-switch.kicad_pcb (KiCad board)
At the start: 2 copper layers, 25.4 x 25.4 mm, 7 parts, among them J1 Conn_01x02_Male, J2 Conn_01x02_Male, J3 Conn_01x02_Male, Q1 AO3401A, Q2 AO3402

Commit message: update to new KiCad format
Other:
- net class Default removed
